Commit message: PSC - Rousselot Otzenberger Blanc Chol Cordelle

File: aida_env/urdf/aida.urdf (robot description, URDF)
Before this commit: robot aida, 33 links, 32 joints
Links:
- link asus_camera_link: mass None -> 0
- link asus_camera_link_optical: mass None -> 0
- link base_laser: mass None -> 0
- link base_link: mass None -> 10
- link nav_module_link: mass None -> 0
- link rgb_cam_rl_link: mass None -> 0
- link rgb_cam_rr_link: mass None -> 0
Joints:
- joint left_front_foot_hinge: origin xyz=0.3 0 0 rpy=0 0 0 -> xyz=0.3 0 0.1 rpy=0 0 0
- joint left_rear_foot_hinge: origin xyz=0.3 0 0 rpy=0 0 0 -> xyz=0.3 0 0.1 rpy=0 0 0
- joint right_front_foot_hinge: origin xyz=0.3 0 0 rpy=0 0 0 -> xyz=0.3 0 0.1 rpy=0 0 0
- joint right_rear_foot_hinge: origin xyz=0.3 0 0 rpy=0 0 0 -> xyz=0.3 0 0.1 rpy=0 0 0
